File: robot_driver_mk1.kicad_sch (KiCad schematic)
At the start: 18 parts, among them J1 Conn_01x03, J10 Conn_01x04, J2 Conn_01x10, J3 Conn_01x04, J4 Conn_01x04, J5 Conn_01x04, J6 Conn_01x04, J7 Conn_01x04, J8 Conn_01x04, J9 Conn_01x04, M1 Stepper_Motor_bipolar, M2 Stepper_Motor_bipolar, M3 Stepper_Motor_bipolar, M4 Stepper_Motor_bipolar, U1 STK672-080-E, U2 STK672-080-E, U3 STK672-080-E, U4 STK672-080-E

Commit message: version mk1.1.1
Parts:
- added D1, D2, D3, D4, D5, D6, D7, D8: LED, symbol Device:LED
- added J11, J12, J16: Conn_01x08, symbol Connector_Generic:Conn_01x08
- added J13, J17: Conn_01x09, symbol Connector_Generic:Conn_01x09
- added J14, J15, J18, J19: Conn_01x03, symbol Connector_Generic:Conn_01x03
- added M5, M6: Motor_Servo, symbol Motor:Motor_Servo
- added R1, R2, R3, R4, R5, R6, R7, R8: R, symbol Device:R
- added SW1, SW2, SW3, SW4, SW5, SW6, SW7, SW8: SW_Push_Open, symbol Switch:SW_Push_Open
Connections:
- net GND: now also J12.3 (Pin_3), J14.3 (Pin_3), J15.3 (Pin_3), J16.8 (Pin_8)
- net VCC: now also J16.1 (Pin_1)
- net PWM: now reaches J2.2 (Pin_2), U1.11 (CLOCK)
- net PWM: now also J2.3 (Pin_3), U2.11 (CLOCK)
- net VCTRL renamed +5V
- net +5V: now also J14.2 (Pin_2), J15.2 (Pin_2), J16.2 (Pin_2)
- new net: J19.1 (Pin_1), M6.1 (PWM)
- new net: J19.2 (Pin_2), M6.2 (+)
- new net: J19.3 (Pin_3), M6.3 (-)
- new net: J17.2 (Pin_2), SW1.1 (A)
- new net: D6.1 (K), J11.3 (Pin_3)
- new net: D6.2 (A), R3.1
- new net: D5.2 (A), R1.1
- new net: J13.2 (Pin_2), R1.2
- new net: J17.3 (Pin_3), SW2.1 (A)
- new net: J17.4 (Pin_4), SW3.1 (A)
- new net: J17.5 (Pin_5), SW4.1 (A)
- new net: J18.1 (Pin_1), M5.1 (PWM)
- new net: J18.2 (Pin_2), M5.2 (+)
- new net: J18.3 (Pin_3), M5.3 (-)
- new net: J17.9 (Pin_9), SW8.1 (A)
- new net: D7.1 (K), J11.5 (Pin_5)
- new net: D7.2 (A), R5.1
- new net: D8.2 (A), R7.1
- new net: J13.8 (Pin_8), R7.2
- new net: D4.1 (K), J11.8 (Pin_8)
- new net: D4.2 (A), R8.1
- new net: J17.6 (Pin_6), SW5.1 (A)
- new net: J17.7 (Pin_7), SW6.1 (A)
- new net: D5.1 (K), J11.1 (Pin_1)
- new net: D1.1 (K), J11.2 (Pin_2)
- new net: D2.1 (K), J11.4 (Pin_4)
- new net: D3.1 (K), J11.6 (Pin_6)
- new net: D8.1 (K), J11.7 (Pin_7)
- new net: J13.4 (Pin_4), R3.2
- new net: D2.2 (A), R4.1
- new net: D1.2 (A), R2.1
- new net: J13.3 (Pin_3), R2.2
- new net: J13.5 (Pin_5), R4.2
- new net: D3.2 (A), R6.1
- new net: J13.7 (Pin_7), R6.2
- new net: J17.8 (Pin_8), SW7.1 (A)
- new net: J13.6 (Pin_6), R5.2
- new net: J12.4 (Pin_4), J16.3 (Pin_3)
- new net: J12.5 (Pin_5), J16.4 (Pin_4)
- new net: J12.6 (Pin_6), J16.5 (Pin_5)
- new net: J12.7 (Pin_7), J16.6 (Pin_6)
- new net: J12.8 (Pin_8), J16.7 (Pin_7)
- new net: J13.9 (Pin_9), R8.2
- new net PWM1: J12.1 (Pin_1), J14.1 (Pin_1)
- new net PWM2: J12.2 (Pin_2), J15.1 (Pin_1)
- new net Vref: J13.1 (Pin_1), J17.1 (Pin_1), SW1.2 (B), SW2.2 (B), SW3.2 (B), SW4.2 (B), SW5.2 (B), SW6.2 (B), SW7.2 (B), SW8.2 (B)
Other:
- note added: "11/04/2023"
- note added: "7 GPIO pins"
- note added: "8 GPIO pins"
- note added: "9 GPIO pins"
- note added: "driver unit"
- note added: "measurements and tools supplies"
- note added: "mk1.1.1"
- note added: "motors (external)"
- note added: "note: parts marked as "(external)" are not included in the driver, they visualize the connected parts from the robot"
- note added: "robot driver mk1"
- note added: "robot_controller_mk1"
- note added: "switches and motors (ext)"
- note added: "tool supply"

Commit message: fixing schematic issues
Connections:
- net GND: no longer U1.14 (MOI), U2.14 (MOI), U3.14 (MOI), U4.14 (MOI)
- no-connect marks 0 -> 5
Changed lines of the file:
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@@
 (kicad_sch (version 20211123) (generator eeschema)
   (paper "A4")
-  (junction (at 87.63 148.59) (diameter 0) (color 0 0 0 0)
-  )
   (junction (at 255.27 55.245) (diameter 0) (color 0 0 0 0)
   )
@@
   (junction (at 255.27 45.085) (diameter 0) (color 0 0 0 0)
   )
-  (junction (at 87.63 186.69) (diameter 0) (color 0 0 0 0)
-  )
   (junction (at 72.39 186.69) (diameter 0) (color 0 0 0 0)
   )
@@
   (junction (at 213.36 92.075) (diameter 0) (color 0 0 0 0)
   )
-  (junction (at 87.63 110.49) (diameter 0) (color 0 0 0 0)
-  )
   (junction (at 55.88 110.49) (diameter 0) (color 0 0 0 0)
   )
@@
   (junction (at 42.545 29.845) (diameter 0) (color 0 0 0 0)
   )
-  (junction (at 87.63 72.39) (diameter 0) (color 0 0 0 0)
-  )
   (junction (at 72.39 62.23) (diameter 0) (color 0 0 0 0)
   )
   (junction (at 69.85 135.89) (diameter 0) (color 0 0 0 0)
   )
+  (no_connect (at 102.87 97.79))
+  (no_connect (at 102.87 135.89))
+  (no_connect (at 102.87 173.99))
+  (no_connect (at 127 151.765))
+  (no_connect (at 102.87 59.69))
   (polyline (pts (xy 22.86 15.875) (xy 111.76 15.875))
     (stroke (width 0) (type default) (color 0 0 0 0))
@@
     (stroke (width 0) (type default) (color 0 0 0 0))
   )
-  (wire (pts (xy 87.63 110.49) (xy 102.87 110.49))
-    (stroke (width 0) (type default) (color 0 0 0 0))
-  )
   (polyline (pts (xy 112.395 97.155) (xy 112.395 121.285))
     (stroke (width 0) (type default) (color 0 0 0 0))
@@
     (stroke (width 0) (type default) (color 0 0 0 0))
   )
-  (wire (pts (xy 102.87 148.59) (xy 102.87 135.89))
-    (stroke (width 0) (type default) (color 0 0 0 0))
-  )
   (wire (pts (xy 201.295 111.76) (xy 218.44 111.76))
     (stroke (width 0) (type default) (color 0 0 0 0))
@@
     (stroke (width 0) (type default) (color 0 0 0 0))
   )
-  (wire (pts (xy 102.87 72.39) (xy 102.87 59.69))
-    (stroke (width 0) (type default) (color 0 0 0 0))
-  )
   (wire (pts (xy 236.22 79.375) (xy 241.3 79.375))
     (stroke (width 0) (type default) (color 0 0 0 0))
@@
     (stroke (width 0) (type default) (color 0 0 0 0))
   )
-  (wire (pts (xy 87.63 186.69) (xy 102.87 186.69))
-    (stroke (width 0) (type default) (color 0 0 0 0))
-  )
   (polyline (pts (xy 155.575 189.865) (xy 155.575 15.875))
     (stroke (width 0) (type default) (color 0 0 0 0))
@@
     (stroke (width 0) (type default) (color 0 0 0 0))
   )
-  (wire (pts (xy 102.87 186.69) (xy 102.87 173.99))
-    (stroke (width 0) (type default) (color 0 0 0 0))
-  )
   (wire (pts (xy 74.93 80.01) (xy 72.39 80.01))
     (stroke (width 0) (type default) (color 0 0 0 0))
@@
     (stroke (width 0) (type default) (color 0 0 0 0))
   )
-  (wire (pts (xy 102.87 110.49) (xy 102.87 97.79))
-    (stroke (width 0) (type default) (color 0 0 0 0))
-  )
   (wire (pts (xy 129.54 161.29) (xy 129.54 154.305))
     (stroke (width 0) (type default) (color 0 0 0 0))
@@
     (stroke (width 0) (type default) (color 0 0 0 0))
   )
-  (wire (pts (xy 87.63 148.59) (xy 102.87 148.59))
-    (stroke (width 0) (type default) (color 0 0 0 0))
-  )
   (wire (pts (xy 122.555 125.73) (xy 132.08 125.73))
     (stroke (width 0) (type default) (color 0 0 0 0))
@@
     (stroke (width 0) (type default) (color 0 0 0 0))
   )
-  (wire (pts (xy 87.63 72.39) (xy 102.87 72.39))
-    (stroke (width 0) (type default) (color 0 0 0 0))
-  )
